File: Hardware/SH002.kicad_pcb (KiCad board)
At the start: 2 copper layers, 100 x 102.5 mm, 247 parts, among them CN1 HX JN1.27-2X5 TP H4.9, CN2 HX JN1.27-2X5 TP H4.9, J10 Conn_01x03, J11 Conn_01x03, J12 Conn_01x03, J13 Conn_01x02, J14 Conn_01x04, J3 Conn_01x04, J4 Conn_01x02, J5 Conn_01x04, J6 Conn_01x03, J7 Conn_01x04, J8 Conn_01x02, J9 Conn_01x02, Q1 2N7002K, Q2 2N7002K, SW1 SW_DIP_x04, U1 ESP32-C3-WROOM-02, U19 SP3485EN, U20 AT24C256C, U22 MCU, STM32G0B0CETx, U3 TLV62080DSGR, U4 RT7272BGSP, U5 TPS259260DRCR

Commit message: remove unused sheets
Parts:
- removed C14: 2.7nF, PCM_JLCPCB:C_0603
- removed C2, C38, C5: 100nF, PCM_JLCPCB:C_0603
- removed C29, C32, C33, C34, C35: 100nF, PCM_JLCPCB:C_0805
- removed C3: 10uF, PCM_JLCPCB:C_0603
- removed C36, C37, C39: 16V 100uF, EasyEDA:CAP-SMD_BD6.3-L6.6-W6.6-LS7.2-FD
- removed C4: 1uF, PCM_JLCPCB:C_0603
- removed C46: 22uF, PCM_JLCPCB:C_0805
- removed C8: CL21A475KBQNNNE, PCM_JLCPCB:C_0805
- removed CN1, CN2: HX JN1.27-2X5 TP H4.9, EasyEDA:IDC-TH_10P-P1.27-V-M-R2-C5-S1.27
- removed D31, D32, D33, D34: LED, LED_THT:LED_D3.0mm
- removed D36: 1N4001W, PCM_JLCPCB:D_SOD-123FL
- removed D39, D8: BZV55B3V6, Diode_SMD:D_MiniMELF
- removed D4: SMAJ28CA, PCM_JLCPCB:D_SMA
- removed F10, F11, F5, F6, F7, F8, F9: JK-NSMD012, EasyEDA:F1206
- removed F16: ASMD1206-200-16V, EasyEDA:F1206
- removed F18: Fuse, Resistor_SMD:R_1812_4532Metric_Pad1.30x3.40mm_HandSolder
- removed J10, J11, J12: Conn_01x03, EASYEDA2KICAD:PhoenixContact_MC_1,5_3-G-3.81_1x03_P3.81mm_Horizontal
- removed J13, J8, J9: Conn_01x02, EASYEDA2KICAD:PhoenixContact_MC_1,5_2-G-3.81_1x02_P3.81mm_Horizontal
- removed J14: Conn_01x04, Connector_Molex:Molex_KK-254_AE-6410-04A_1x04_P2.54mm_Vertical
- removed J7: Conn_01x04, EASYEDA2KICAD:PhoenixContact_MC_1,5_4-G-3.81_1x04_P3.81mm_Horizontal
- removed L1: IND, 6.8uH 2.8A, PCM_JLCPCB:IND-SMD_L4.0-W4.0
- removed L4: SMCM9070-701T, EasyEDA:FILTER-SMD_4P-L9.0-W7.0-LS9.5-1
- removed LCD1: ST7735 1.8in SPI, EASYEDA2KICAD:LCD, ST7735 1.8in SPI
- removed LCD5: ST7735 2.8in SPI, AderbTech:LCD 2.8 INCH SPI ST7735
- removed R105, R106, R107, R108, R109, R110, R111, R34, R35, R36, R37, R38, R39, R40, R41, R5, R61: 10kΩ, PCM_JLCPCB:R_0603
- removed R117, R118, R22, R23, R24, R25, R30, R32, R33, R42, R43, R44, R45, R46, R47, R48, R53: HMLV1812-470G, Resistor_SMD:R_1812_4532Metric_Pad1.30x3.40mm_HandSolder
- removed R119: 33kΩ, PCM_JLCPCB:R_0603
- removed R12, R16, R18, R20, R8: 1kΩ, PCM_JLCPCB:R_0805
- removed R15, R17, R19, R21: 10kΩ, PCM_JLCPCB:R_0805
- removed R25, R54: 100kΩ, PCM_JLCPCB:R_0603
- removed R26, R27, R28, R29: 5.1kΩ, PCM_JLCPCB:R_0603
- removed R4, R56: 330Ω, PCM_JLCPCB:R_0603
- removed R62: 49.9Ω, PCM_JLCPCB:R_0603
- removed R92: 12kΩ, PCM_JLCPCB:R_0603
- removed R93, R94, R95, R96, R97, R98, R99: 3.3kΩ, PCM_JLCPCB:R_0603
- removed S1: Tactile Button, 160gf, PCM_JLCPCB:SW_TS-1088-AR02016
- removed SW1: SW_DIP_x04, Button_Switch_THT:SW_DIP_SPSTx04_Slide_9.78x12.34mm_W7.62mm_P2.54mm
- removed TP1, TP2, TP3, TP4, TP5, TP6, TP7: TestPoint, TestPoint:TestPoint_Pad_D1.0mm
- removed U1: ESP32-C3-WROOM-02, RF_Module:ESP32-C3-WROOM-02
- removed U5: TPS259260DRCR, EasyEDA:VSON-10_L3.0-W3.0-P0.50-TL-EP-1
- added BZ2: SMD-8503-3627-16Ω, EasyEDA:BUZ-SMD_4P-L8.5-W8.5-BR-1, F.Cu at (90.8, 125.6)
- added C11: 22uF, PCM_JLCPCB:C_0805, F.Cu at (123.1, 64.7)
- added D18: P0640SCLRP, EasyEDA:SMB_L4.6-W3.6-LS5.3-BI, F.Cu at (147.2, 53.4)
- added D19: P0640SCLRP, EasyEDA:SMB_L4.6-W3.6-LS5.3-BI, F.Cu at (110.3, 60.9)
- added D3: NH-Z3535RGBA-SG, EasyEDA:LED-ARRAY-SMD_6P-L3.7-W3.5-TL-RD, F.Cu at (90.0, 73.8)
- added FL1: ACM70V-701-2PL-TL00, EasyEDA:FILTER-SMD_4P-L7.0-W6.0-TL_ACM70V, F.Cu at (128.4, 54.1)
- added J1: Conn_01x07, AderbTech:Keypad_3X4, F.Cu at (123.1, -13.1)
- added J2: Connector, USB-TYPE-C-16P, EasyEDA:IDC-SMD_10P-P1.27-3220-10-0300-00, F.Cu at (122.5, 135.0)
- added R75: 10kΩ, PCM_JLCPCB:R_0603, F.Cu at (155.6, 71.6)
- added R84: 10kΩ, PCM_JLCPCB:R_0603, F.Cu at (155.6, 73.8)
- added R85: 10kΩ, PCM_JLCPCB:R_0603, F.Cu at (155.6, 76.1)
- added RN10: 4D03WGJ0471T5E, EasyEDA:RES-ARRAY-SMD_0603-8P-L3.2-W1.6-BL, F.Cu at (96.2, 73.8)
- added RN11: 4D03WGJ0471T5E, EasyEDA:RES-ARRAY-SMD_0603-8P-L3.2-W1.6-BL, F.Cu at (96.2, 106.2)
- added RN9: 4D03WGJ0471T5E, EasyEDA:RES-ARRAY-SMD_0603-8P-L3.2-W1.6-BL, F.Cu at (96.2, 90.0)
- added SW2: RotaryEncoder_Switch_MP, Rotary_Encoder:RotaryEncoder_Alps_EC11E-Switch_Vertical_H20mm, F.Cu at (141.2, 115.0)
- added U2: TPS259251DRCR, EasyEDA:WSON-10_L3.0-W3.0-P0.50-BL-EP, F.Cu at (128.4, 60.2)
- BAT1: footprint EasyEDA:BAT-SMD_796136-1 -> EASYEDA2KICAD:BAT-SMD_796136-1
- C10: value 100nF -> 22uF; footprint PCM_JLCPCB:C_0603 -> PCM_JLCPCB:C_0805
- C31: value 100nF -> 4.7nF; footprint PCM_JLCPCB:C_0805 -> PCM_JLCPCB:C_0603
- C7: value 10uF -> 100nF; footprint PCM_JLCPCB:C_0805 -> PCM_JLCPCB:C_0603
- C9: value 1uF -> 22uF; footprint PCM_JLCPCB:C_0603 -> PCM_JLCPCB:C_0805
- D1, D2: value LED -> NH-Z3535RGBA-SG; footprint LED_THT:LED_D3.0mm -> EasyEDA:LED-ARRAY-SMD_6P-L3.7-W3.5-TL-RD
- D11: value BZV55B3V6 -> 1N4001W; footprint Diode_SMD:D_MiniMELF -> PCM_JLCPCB:D_SOD-123FL
- D12, D9: value BZV55B3V6 -> P0640SCLRP; footprint Diode_SMD:D_MiniMELF -> EasyEDA:SMB_L4.6-W3.6-LS5.3-BI
- D15: value BZV55B3V6 -> Red; footprint Diode_SMD:D_MiniMELF -> PCM_JLCPCB:D_0603
- D16: value SMAJ28CA -> SMF5.0A; footprint PCM_JLCPCB:D_SMA -> PCM_JLCPCB:D_SOD-123FL
- D17: value Red -> SMF5.0A; footprint PCM_JLCPCB:D_0603 -> PCM_JLCPCB:D_SOD-123FL
- D6, D7: value BZV55B3V6 -> SMF12A; footprint Diode_SMD:D_MiniMELF -> PCM_JLCPCB:D_SOD-123FL
- F1: value ASMD1206-200-16V -> MF-MSMF110/16-2; footprint EasyEDA:F1206 -> Fuse:Fuse_1812_4532Metric_Pad1.30x3.40mm_HandSolder
- F19, F2, F3, F4: footprint EasyEDA:F1206 -> EASYEDA2KICAD:F1206
- J5: value Conn_01x04 -> Conn_01x02; footprint EASYEDA2KICAD:PhoenixContact_MC_1,5_4-G-3.81_1x04_P3.81mm_Horizontal -> EASYEDA2KICAD:PhoenixContact_MC_1,5_2-G-3.81_1x02_P3.81mm_Horizontal
- J6: value Conn_01x03 -> Conn_01x02; footprint EASYEDA2KICAD:PhoenixContact_MC_1,5_3-G-3.81_1x03_P3.81mm_Horizontal -> EASYEDA2KICAD:PhoenixContact_MC_1,5_2-G-3.81_1x02_P3.81mm_Horizontal
- L3: value ACM70V-701-2PL-TL00 -> L; footprint EasyEDA:FILTER-SMD_4P-L7.0-W6.0-TL_ACM70V -> Inductor_SMD:L_Coilcraft_1008HQ_2520Metric
- LCD2: value Conn_01x04 -> 20X4 I2C
- LCD3: value ST7735 2.8in SPI -> ST7735 2.79in SPI; footprint AderbTech:LCD 2.8 INCH SPI HEADER -> AderbTech:LCD 2.79 INCH SPI HEADER NMH
- LCD4: value ST7735 1.9in SPI -> ST7735 2.79in SPI; footprint AderbTech:LCD 1.9 INCH SPI ST7735 -> AderbTech:LCD 2.79 INCH SPI ST7789
- R10: value 1kΩ -> 33kΩ; footprint PCM_JLCPCB:R_0805 -> PCM_JLCPCB:R_0603
- R11: value 10kΩ -> 47kΩ; footprint PCM_JLCPCB:R_0805 -> PCM_JLCPCB:R_0603
- R13: value 10kΩ -> 1MΩ; footprint PCM_JLCPCB:R_0805 -> PCM_JLCPCB:R_0603
- R14: value 1kΩ -> 330kΩ; footprint PCM_JLCPCB:R_0805 -> PCM_JLCPCB:R_0603
- R2, R72, R73: value 330Ω -> 49.9Ω
- R3: value 330Ω -> 10kΩ
- R9: value 10kΩ -> 100kΩ; footprint PCM_JLCPCB:R_0805 -> PCM_JLCPCB:R_0603
- R91: value 56kΩ -> 49.9Ω
- U4: value RT7272BGSP -> AP63357DV-7; footprint Package_SO:SOIC-8-1EP_3.9x4.9mm_P1.27mm_EP2.29x3mm -> EASYEDA2KICAD:V-DFN3020-13-A_L3.0-W2.0-P0.45-BL-EP_AP6335X
- moved LCD3 174.9 mm to (108.8, 126.2), turned to 90 degrees
- moved TP12 132.0 mm to (184.4, 63.0)
- moved H3 128.1 mm to (155.0, 45.0)
- moved H1 114.9 mm to (155.0, 135.0)
- moved J6 100.1 mm to (101.9, 45.0), turned to 180 degrees
- moved TP16 93.4 mm to (166.2, 43.1)
- moved C41 91.9 mm to (139.4, 66.9), turned to 90 degrees
- moved R80 91.6 mm to (109.4, 111.2)
- moved R86 90.0 mm to (135.6, 73.8), turned to -90 degrees
- moved R79 89.7 mm to (109.4, 109.4)
- moved R88 89.1 mm to (135.6, 70.2)
- moved C40 88.3 mm to (137.5, 66.9), turned to 90 degrees
- moved U3 88.1 mm to (133.3, 70.3), turned to 90 degrees
- moved D14 87.9 mm to (137.5, 63.0), turned to 90 degrees
- moved R49 86.7 mm to (135.6, 62.9), turned to 90 degrees
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Connections:
- net /OUTPUTS/EXT_LED renamed /PGM/EXT_LED
- net /RS485/485_DE_~{RE} renamed /EXPANSION/485_DE_~{RE}
- net /RS485/485_RX renamed /EXPANSION/485_RX
- net /RS485/485_TX renamed /EXPANSION/485_TX
- net /ZONES_8W/ADC_ZONE/ADC_RAW renamed /ADC_ZONE/ADC_RAW
- C1 pad 1: /STATUS_LED/USER_BTN -> /LED_STATUS/USER_BTN
- C10 pad 1: +3V3 -> +VSYS
- C12 pad 1: Net-(U4-BOOT) -> Net-(U4-BST)
- C12 pad 2: /POWER/SW -> /POWER/PWR_5V0/SW
- C28 pad 1: Net-(D39-K) -> Net-(C28-Pad1)
- C30 pad 1: Net-(D7-K) -> VPROT
- C31 pad 1: Net-(D8-K) -> Net-(U2-dV/dT)
- C7 pad 1: +VSYS -> /POWER/VSYS_ADC
- C9 pad 1: +3V3 -> +VSYS
- D1 pad 2: Net-(D1-A) -> GND
- D10 pad 1: Net-(D10-K) -> /ADC_ZONE/ADC_MCU
- D11 pad 1: Net-(D11-K) -> +3V3
- D11 pad 2: GND -> Net-(BZ2-Pad2)
- D12 pad 1: Net-(D12-K) -> GND
- D12 pad 2: GND -> /EXPANSION/485_N
- D15 pad 1: /POWER/VSYS_ADC -> GND
- D15 pad 2: GND -> Net-(D15-Pad2)
- D16 pad 1: GND -> Net-(D16-Pad1)
- D16 pad 2: /POWER/PWR_RAW -> GND
- D17 pad 1: Net-(D17-Pad1) -> /POWER/VSYS_ADC
- D17 pad 2: +VSYS -> GND
- D2 pad 2: Net-(D2-A) -> GND
- D37 pad 2: /OUTPUTS/EXT_LED_RTN -> /PGM/EXT_LED_RTN
- D38 pad 1: /RS485/485_P -> /EXPANSION/485_P
- D38 pad 2: /RS485/485_N -> /EXPANSION/485_N
- D6 pad 1: Net-(D6-K) -> VPROT
- D7 pad 1: Net-(D7-K) -> +VSYS
- D9 pad 1: Net-(D9-K) -> PWR-
- D9 pad 2: GND -> PWR+
- F1 pad 1: /VCOM -> Net-(F1-Pad1)
- F1 pad 2: +VSYS -> PWR+
- F19 pad 1: +5V0 -> +VSYS
- F2 pad 1: /OUTPUTS/EXT_LED_RTN -> /PGM/EXT_LED_RTN
- F3 pad 1: /OUTPUTS/SIREN_RTN -> Net-(BZ2-Pad2)
- F4 pad 1: Net-(D39-K) -> Net-(D16-Pad1)
- J3 pad 1: /RS485/485_P -> /EXPANSION/485_P
- J3 pad 2: /RS485/485_N -> /EXPANSION/485_N
- J3 pad 3: GND -> PWR-
- J3 pad 4: /VCOM -> PWR+
- J4 pad 1: PWR+ -> PWR-
- J4 pad 2: PWR- -> PWR+
- J5 pad 1: /RS485/485_P -> +VSYS
- J5 pad 2: /RS485/485_N -> /PGM/EXT_LED_RTN
- L3 pad 1: unconnected-(L3-Pad1) -> /POWER/PWR_5V0/SW
- L3 pad 2: unconnected-(L3-Pad2) -> +5V0
- LCD2 pad 1: +3V3 -> /ST7735/LCD_SDA
- LCD2 pad 2: /SDA -> /ST7735/LCD_SCL
- LCD2 pad 3: /SCL -> +3V3
- LCD3 pad 1: unconnected-(LCD3-GND-Pad1) -> /ST7735/LCD_BL
- LCD3 pad 2: unconnected-(LCD3-VCC-Pad2) -> /ST7735/LCD_CS
- LCD3 pad 3: unconnected-(LCD3-SCL-Pad3) -> /ST7735/LCD_DC
- LCD3 pad 4: unconnected-(LCD3-SDA-Pad4) -> /ST7735/LCD_RST
- LCD3 pad 5: unconnected-(LCD3-FD-Pad5) -> Net-(LCD3-SDA)
- LCD3 pad 6: unconnected-(LCD3-DC-Pad6) -> Net-(LCD3-SCL)
- LCD3 pad 7: unconnected-(LCD3-CS-Pad7) -> +3V3
- LCD3 pad 8: unconnected-(LCD3-BLK-Pad8) -> GND
- R1 pad 1: Net-(D17-Pad1) -> +VSYS
- R1 pad 2: GND -> Net-(D15-Pad2)
- R10 pad 1: Net-(R10-Pad1) -> /POWER/VSYS_ADC
- R10 pad 2: Net-(D7-K) -> GND
- R104 pad 1: /STM32/PA02 -> /ADC_ZONE/ADC_MCU
- R11 pad 1: +VADC -> Net-(U2-ILIM)
- R11 pad 2: Net-(D7-K) -> GND
- R116 pad 1: /STM32/PA02 -> /ADC_ZONE/ADC_MCU
- R116 pad 2: Net-(R116-Pad2) -> Net-(C28-Pad1)
- R13 pad 1: +VADC -> VPROT
- R13 pad 2: Net-(D8-K) -> Net-(U2-EN/UVLO)
- R14 pad 1: Net-(R108-Pad2) -> Net-(U2-EN/UVLO)
- R14 pad 2: Net-(D9-K) -> GND
- R2 pad 1: Net-(D31-A) -> /BUZZER/BUZZ
- R2 pad 2: /STATUS_LED/LED_TRIP -> Net-(Q1-G)
- R3 pad 1: Net-(D32-A) -> Net-(Q1-G)
- R3 pad 2: /STATUS_LED/LED_FAULT -> GND
- R31 pad 2: /OUTPUTS/EXT_LED_RTN -> /PGM/EXT_LED_RTN
- R57 pad 2: /STATUS_LED/USER_BTN -> /LED_STATUS/USER_BTN
- R63 pad 1: Net-(LCD1-Pin_3) -> Net-(LCD3-SDA)
- R64 pad 2: Net-(LCD1-Pin_4) -> Net-(LCD3-SCL)
- R65 pad 2: Net-(LCD1-Pin_4) -> Net-(LCD3-SDA)
- R66 pad 2: Net-(LCD1-Pin_3) -> /ST7735/LCD_CS
- R67 pad 2: /ST7735/LCD_CS -> Net-(LCD3-SCL)
- R69 pad 1: Net-(R116-Pad2) -> Net-(C28-Pad1)
- R69 pad 2: Net-(D39-K) -> Net-(D16-Pad1)
- R70 pad 2: /SCL -> /AW21024/AW_SCL
- R71 pad 2: /SDA -> /AW21024/AW_SDA
- R72 pad 1: Net-(D1-A) -> /LED_STATUS/USER_EC1
- R72 pad 2: /STATUS_LED/LED_LINK -> Net-(R72-Pad2)
- R73 pad 1: Net-(D2-A) -> Net-(R73-Pad1)
- R73 pad 2: /STATUS_LED/LED_ACT -> /LED_STATUS/USER_EC2
- R76 pad 1: /RS485/485_N -> /EXPANSION/485_N
- R76 pad 2: /RS485/485_P -> /EXPANSION/485_P
- R77 pad 1: /RS485/485_N -> /EXPANSION/485_N
- R78 pad 2: /RS485/485_P -> /EXPANSION/485_P
- R83 pad 2: Net-(D39-K) -> Net-(D16-Pad1)
- R9 pad 1: +VADC -> +VSYS
- R9 pad 2: Net-(D6-K) -> /POWER/VSYS_ADC
- R91 pad 1: Net-(U4-RLIM) -> Net-(R75-Pad2)
- R91 pad 2: GND -> /LED_STATUS/USER_EC_BTN
- S2 pad 2: /STATUS_LED/USER_BTN -> /LED_STATUS/USER_BTN
- TP13 pad 1: /SCL -> /AW21024/AW_SCL
- TP14 pad 1: /SDA -> /AW21024/AW_SDA
- TP22 pad 1: Net-(R116-Pad2) -> Net-(C28-Pad1)
- U19 pad 6: /RS485/485_P -> /EXPANSION/485_P
- U19 pad 7: /RS485/485_N -> /EXPANSION/485_N
- U20 pad 5: /SDA -> /AW21024/AW_SDA
- U20 pad 6: /SCL -> /AW21024/AW_SCL
- U22 pad 1: /ESP_EN -> /STM32/PC13
- U22 pad 11: /EXP_ADDR/485_ADC_ADDR -> /STM32/PA00
- U22 pad 14: /STM32/PA03 -> /KEYPAD/KEY_C1
- U22 pad 17: /STM32/PA06 -> /KEYPAD/KEY_C2
- U22 pad 18: /STM32/PA07 -> /KEYPAD/KEY_R4
- U22 pad 19: /STM32/PB00 -> /KEYPAD/KET_C3
- U22 pad 20: /STM32/PB01 -> /KEYPAD/KEY_R1
- U22 pad 21: /STM32/PB02 -> /KEYPAD/KEY_R2
- U22 pad 22: /STM32/PB10 -> /KEYPAD/KEY_R3
- U22 pad 25: /STATUS_LED/USER_BTN -> /LED_STATUS/LED_CONFIG
- U22 pad 26: /STATUS_LED/LED_TRIP -> /LED_STATUS/LED_RUN
- U22 pad 27: /STATUS_LED/LED_CONFIG -> /LED_STATUS/LED_LINK
- U22 pad 28: /STATUS_LED/LED_FAULT -> /LED_STATUS/LED_ACT
- U22 pad 29: /STATUS_LED/LED_RUN -> /LED_STATUS/LED_ARMED
- U22 pad 30: /STATUS_LED/LED_ACT -> /LED_STATUS/LED_TRIP
- U22 pad 31: /STATUS_LED/LED_LINK -> /LED_STATUS/USER_BTN
- U22 pad 33: /SCL -> /AW21024/AW_SCL
- U22 pad 34: /SDA -> /AW21024/AW_SDA
- U22 pad 38: /OUTPUTS/SIREN -> /BUZZER/BUZZ
- U22 pad 47: /ESP32C3/ESP_IO7 -> /STM32/PB08
- U22 pad 48: /ESP32C3/ESP_IO6 -> /STM32/PB09
- U4 pad 1: /POWER/SW -> +VSYS
- U4 pad 2: Net-(U4-BOOT) -> Net-(U4-EN)
- U4 pad 3: Net-(U4-EN) -> Net-(U4-FB)
- U4 pad 5: Net-(U4-FB) -> unconnected-(U4-PG-Pad5)
- U4 pad 6: Net-(U4-COMP) -> Net-(U4-BST)
- U4 pad 7: Net-(U4-RLIM) -> /POWER/PWR_5V0/SW
- U4 pad 8: +VSYS -> GND
- U4 pad 9: GND -> /POWER/PWR_5V0/SW
Routing:
- net +VSYS: track 155.5 -> 39.3 mm, vias 1 -> 0
- net +3V3: track 129.0 -> 22.8 mm, vias 13 -> 1
- net +VADC: track 71.0 -> 8.07 mm, vias 7 -> 0
- net /ZONES_8W/VSYS_EXT1: track 62.3 -> 0.00 mm
- net /ZONES_8W/ADC_ZONE7/ADC_RAW: track 51.0 -> 0.00 mm
- net /ZONES_8W/ADC_ZONE6/ADC_RAW: track 51.0 -> 0.00 mm
- net /ZONES_8W/ADC_ZONE5/ADC_RAW: track 51.0 -> 0.00 mm
- net /ZONES_8W/ADC_ZONE4/ADC_RAW: track 51.0 -> 0.00 mm
- net /ZONES_8W/ADC_ZONE3/ADC_RAW: track 51.0 -> 0.00 mm
- net /ZONES_8W/ADC_ZONE2/ADC_RAW: track 51.0 -> 0.00 mm
- net /ZONES_8W/ADC_ZONE1/ADC_RAW: track 51.0 -> 0.00 mm
- net /RS485/485_N: track 48.1 -> 0.00 mm
- net /RS485/485_P: track 46.0 -> 0.00 mm, vias 2 -> 0
- net GND: track 109.5 -> 64.6 mm, vias 243 -> 107
- net /VCOM: track 32.9 -> 0.00 mm, vias 2 -> 0
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- removed copper zone on F.Cu, net GND
Other:
- board size 100 x 102.5 mm -> 75 x 100 mm
- board text added: "ARMED"
- board text added: "COMMS"
- board text added: "DEBUG"
- board text added: "MCU"
- board text added: "STATUS"
- board text added: "USER"
- board text added: "VIN"
- board text added: "ZN1"
- board text removed: "12V0"
- board text removed: "ACT"
- board text removed: "ALARM"
- board text removed: "ALM"
- board text removed: "BAT"
- board text removed: "CONFIG"
- board text removed: "ESP RST"
- board text removed: "ESP32"
- board text removed: "EXP ADDRESS"
- board text removed: "FAULT"
- board text removed: "GND"
- board text removed: "LINK"
- board text removed: "OFF"
- board text removed: "ON"
- board text removed: "PWR"
- board text removed: "RTN"
- board text removed: "RUN"
- board text removed: "RXD"
- board text removed: "STM32"
- board text removed: "TXD"
- board text removed: "USR BTN"
- board text removed: "VEXT"
- board text removed: "Z1"
- board text removed: "Z2"
- board text removed: "Z3"
- board text removed: "Z4"
- board text removed: "Z5"
- board text removed: "Z6"
- board text removed: "Z7"
- board text removed: "Z8"
